Commit message: corrected urdf for zero initial angles

File: arm_assembly/urdf/arm_assembly.urdf (robot description, URDF)
Before this commit: robot arm_assembly, 6 links, 5 joints
Links:
- link arm1_link: mass 0.0659056350151723 -> 0.0659056350151601
- link arm2_link: mass 0.0939634786908005 -> 0.0939634772458711
- link arm3_link: mass 0.0234826216736623 -> 0.0234826220419238
Joints:
- joint joint1: origin xyz=0 0 0 rpy=0 0 0 -> xyz=-0.0012854 0.004 0.020614 rpy=0 0 0
- joint joint2: origin xyz=0.013919 0 0.040276 rpy=0 0 0 -> xyz=0.015204 0 0.019662 rpy=0 0 0
- joint joint3: origin xyz=0 0 0.12 rpy=0 -0.0085284 0 -> xyz=0 0 0.12 rpy=0 0 0
- joint joint4: origin xyz=-0.0053 0.011 0.093753 rpy=0 0 0 -> xyz=-0.0053 0.007 0.09375 rpy=0 0 0
- joint joint5: origin xyz=-0.005 0 0.027997 rpy=0 0 0 -> xyz=-0.005 0 0.028 rpy=0 0 0
